File: kicad/photoacoustic-detector.kicad_pcb (KiCad board)
At the start: 2 copper layers, 22.8 x 53.4 mm, 17 parts, among them J1 527450697, U1 TLV320ADC6120IRTER, U2 RP-PICO-H

Commit message: micropython code
Parts:
- moved C2 2.35 mm to (167.1, 93.6)
- moved C1 1.87 mm to (169.3, 93.6)
- moved J1 1.37 mm to (168.6, 99.9), turned to 0 degrees
- moved C3 0.21 mm to (168.2, 93.6)
Routing:
- net Net-(C3-Pad1): track 7.00 -> 4.06 mm
- net Net-(C2-Pad1): track 7.20 -> 4.33 mm
- net MICBIAS: track 22.1 -> 19.3 mm
- net OUT-: track 7.12 -> 5.92 mm
- net GND: track 0.00 -> 0.97 mm, vias 2 -> 3
- net OUT+: track 7.62 -> 7.92 mm, vias 0 -> 2

Commit message: updated the kicad and added the pc-gui
Parts:
- J1: value 527450697 -> 527450897; footprint Personal_Library:CON_527450697_MOL -> Personal_Library_local:CONN_527450897_MOL
- moved C1 2.54 mm to (171.7, 94.3)
- moved C3 1.77 mm to (169.8, 94.3)
- moved C10 1.42 mm to (173.6, 86.0)
- moved C11 1.42 mm to (173.6, 87.0)
- moved J1 1.38 mm to (170.0, 99.6)
- moved C2 1.32 mm to (168.2, 94.2)
Connections:
- J1 pad 1: unconnected-(J1-Pad1) -> GND
- J1 pad 2: unconnected-(J1-Pad2) -> GND
Routing:
- net SDOUT: track 23.8 -> 26.4 mm
- net Net-(J1-Pin_5): track 4.06 -> 1.60 mm
- net DREG: track 2.61 -> 4.70 mm
- net OUT+: track 7.92 -> 9.84 mm
- net Net-(J1-Pin_4): track 4.33 -> 2.50 mm
- net OUT-: track 5.92 -> 7.37 mm
- net BCLK: track 27.9 -> 29.4 mm
- net GND: track 0.97 -> 0.00 mm, vias 3 -> 2
Other:
- board text added: "Photoacoustic detector v0.0.2"
- board text removed: "Photoacoustic detector v0.0.1"
