File: kicad/photoacoustic-detector.kicad_sch (KiCad schematic)
At the start: 17 parts, among them J1 527450697, U1 TLV320ADC6120IRTER, U2 RP-PICO-H

Commit message: micropython code
Parts:
- removed J1: 527450697, Personal_Library:CON_527450697_MOL, symbol Personal_Library:527450697
Changed lines of the file:
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@@
-	)
-	(symbol
-		(lib_id "Personal_Library:527450697")
-		(at 63.5 44.45 0)
-		(unit 1)
-		(body_style 1)
-		(exclude_from_sim no)
-		(in_bom yes)
-		(on_board yes)
-		(in_pos_files yes)
-		(dnp no)
-		(fields_autoplaced yes)
-		(property "Reference" "J1"
-			(at 77.47 52.0699 0)
-			(show_name no)
-			(do_not_autoplace no)
-			(effects
-				(font
-					(size 1.524 1.524)
-				)
-				(justify left)
-			)
-		)
-		(property "Value" "527450697"
-			(at 77.47 54.6099 0)
-			(show_name no)
-			(do_not_autoplace no)
-			(effects
-				(font
-					(size 1.524 1.524)
-				)
-				(justify left)
-			)
-		)
-		(property "Footprint" "Personal_Library:CON_527450697_MOL"
-			(at 63.5 44.45 0)
-			(hide yes)
-			(show_name no)
-			(do_not_autoplace no)
-			(effects
-				(font
-					(size 1.27 1.27)
-					(italic yes)
-				)
-			)
-		)
-		(property "Datasheet" "https://www.molex.com/en-us/products/part-detail-pdf/527450697?display=pdf"
-			(at 63.5 44.45 0)
-			(hide yes)
-			(show_name no)
-			(do_not_autoplace no)
-			(effects
-				(font
-					(size 1.27 1.27)
-					(italic yes)
-				)
-			)
-		)
-		(property "Description" ""
-			(at 63.5 44.45 0)
-			(hide yes)
-			(show_name no)
-			(do_not_autoplace no)
-			(effects
-				(font
-					(size 1.27 1.27)
-				)
-			)
-		)
-		(pin "P1"
-		)
-		(pin "1"
-		)
-		(pin "2"
-		)
-		(pin "3"
-		)
-		(pin "5"
-		)
-		(pin "4"
-		)
-		(pin "6"
-		)
-		(pin "P2"
-		)
-		(instances
-			(project "photoacoustic-detector"
-				(path "/268c6120-58cb-44fb-87db-b7827ba409a7"
-					(reference "J1")
-					(unit 1)
-				)
-			)
-		)
 	)
 	(symbol

Commit message: updated the kicad and added the pc-gui
Parts:
- added J1: 527450897, Personal_Library_local:CONN_527450897_MOL, symbol Connector_Generic:Conn_01x08
Connections:
- net GND: now also J1.1 (Pin_1), J1.2 (Pin_2), J1.7 (Pin_7), J1.8 (Pin_8)
- net MICBIAS: now also J1.6 (Pin_6)
- net at C2.1: now also J1.4 (Pin_4)
- net at C3.1: now also J1.5 (Pin_5)
- no-connect marks 5 -> 3
Changed lines of the file:
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@@
 	(text "IM73A135 flex mic\n"
 		(exclude_from_sim no)
-		(at 53.594 39.624 0)
+		(at 63.754 39.37 0)
 		(effects
 			(font
@@
 	)
 	(junction
-		(at 48.26 62.23)
+		(at 59.69 62.23)
 		(diameter 0)
 		(color 0 0 0 0)
@@
 	)
 	(junction
+		(at 60.96 44.45)
+		(diameter 0)
+		(color 0 0 0 0)
+	)
+	(junction
 		(at 123.19 39.37)
 		(diameter 0)
@@
 	)
 	(no_connect
-		(at 63.5 44.45)
-	)
-	(no_connect
-		(at 63.5 46.99)
-	)
-	(no_connect
 		(at 125.73 69.85)
 	)
@@
 	(wire
 		(pts
+			(xy 60.96 46.99) (xy 60.96 44.45)
+		)
+		(stroke
+			(width 0)
+			(type default)
+		)
+	)
+	(wire
+		(pts
 			(xy 189.23 80.01) (xy 191.77 80.01)
 		)
@@
 	(wire
 		(pts
+			(xy 60.96 44.45) (xy 63.5 44.45)
+		)
+		(stroke
+			(width 0)
+			(type default)
+		)
+	)
+	(wire
+		(pts
 			(xy 48.26 64.77) (xy 48.26 62.23)
 		)
@@
 	(wire
 		(pts
+			(xy 48.26 43.18) (xy 48.26 44.45)
+		)
+		(stroke
+			(width 0)
+			(type default)
+		)
+	)
+	(wire
+		(pts
 			(xy 179.07 106.68) (xy 179.07 109.22)
 		)
@@
 	(wire
 		(pts
-			(xy 124.46 59.69) (xy 125.73 59.69)
+			(xy 63.5 46.99) (xy 60.96 46.99)
 		)
 		(stroke
@@
 	(wire
 		(pts
-			(xy 236.22 60.96) (xy 240.03 60.96)
+			(xy 124.46 59.69) (xy 125.73 59.69)
 		)
 		(stroke
@@
 	(wire
 		(pts
-			(xy 40.64 57.15) (xy 43.18 57.15)
+			(xy 236.22 60.96) (xy 240.03 60.96)
 		)
 		(stroke
@@
 	(wire
 		(pts
-			(xy 191.77 82.55) (xy 191.77 85.09)
+			(xy 40.64 57.15) (xy 43.18 57.15)
 		)
 		(stroke
@@
 	(wire
 		(pts
-			(xy 166.37 106.68) (xy 166.37 109.22)
+			(xy 191.77 82.55) (xy 191.77 85.09)
 		)
 		(stroke
@@
 	(wire
 		(pts
-			(xy 107.95 52.07) (xy 114.3 52.07)
+			(xy 166.37 106.68) (xy 166.37 109.22)
 		)
 		(stroke
@@
 	(wire
 		(pts
-			(xy 48.26 59.69) (xy 63.5 59.69)
+			(xy 107.95 52.07) (xy 114.3 52.07)
 		)
 		(stroke
@@
 	(wire
 		(pts
-			(xy 48.26 62.23) (xy 48.26 59.69)
+			(xy 48.26 44.45) (xy 60.96 44.45)
 		)
 		(stroke
@@
 	(wire
 		(pts
+			(xy 59.69 62.23) (xy 63.5 62.23)
+		)
+		(stroke
+			(width 0)
+			(type default)
+		)
+	)
+	(wire
+		(pts
 			(xy 191.77 87.63) (xy 191.77 85.09)
 		)
@@
 	(wire
 		(pts
+			(xy 63.5 59.69) (xy 59.69 59.69)
+		)
+		(stroke
+			(width 0)
+			(type default)
+		)
+	)
+	(wire
+		(pts
 			(xy 189.23 90.17) (xy 191.77 90.17)
 		)
@@
 	(wire
 		(pts
+			(xy 59.69 59.69) (xy 59.69 62.23)
+		)
+		(stroke
+			(width 0)
+			(type default)
+		)
+	)
+	(wire
+		(pts
 			(xy 171.45 109.22) (xy 171.45 106.68)
 		)
@@
 	(wire
 		(pts
-			(xy 48.26 62.23) (xy 63.5 62.23)
+			(xy 48.26 62.23) (xy 59.69 62.23)
 		)
 		(stroke
@@
 	)
 	(symbol
+		(lib_id "Connector_Generic:Conn_01x08")
+		(at 68.58 52.07 0)
+		(unit 1)
+		(body_style 1)
+		(exclude_from_sim no)
+		(in_bom yes)
+		(on_board yes)
+		(in_pos_files yes)
+		(dnp no)
+		(fields_autoplaced yes)
+		(property "Reference" "J1"
+			(at 71.12 52.0699 0)
+			(show_name no)
+			(do_not_autoplace no)
+			(effects
+				(font
+					(size 1.27 1.27)
+				)
+				(justify left)
+			)
+		)
+		(property "Value" "527450897"
+			(at 71.12 54.6099 0)
+			(show_name no)
+			(do_not_autoplace no)
+			(effects
+				(font
+					(size 1.27 1.27)
+				)
+				(justify left)
+			)
+		)
+		(property "Footprint" "Personal_Library_local:CONN_527450897_MOL"
+			(at 68.58 52.07 0)
+			(hide yes)
+			(show_name no)
+			(do_not_autoplace no)
+			(effects
+				(font
+					(size 1.27 1.27)
+				)
+			)
+		)
+		(property "Datasheet" "https://www.digikey.com/en/products/detail/molex/0527450897/2421443"
+			(at 68.58 52.07 0)
+			(hide yes)
+			(show_name no)
+			(do_not_autoplace no)
+			(effects
+				(font
+					(size 1.27 1.27)
+				)
+			)
+		)
+		(property "Description" "Generic connector, single row, 01x08, script generated (kicad-library-utils/schlib/autogen/connector/)"
+			(at 68.58 52.07 0)
+			(hide yes)
+			(show_name no)
+			(do_not_autoplace no)
+			(effects
+				(font
+					(size 1.27 1.27)
+				)
+			)
+		)
+		(pin "7"
+		)
+		(pin "4"
+		)
+		(pin "8"
+		)
+		(pin "6"
+		)
+		(pin "2"
+		)
+		(pin "1"
+		)
+		(pin "5"
+		)
+		(pin "3"
+		)
+		(instances
+			(project "photoacoustic-detector"
+				(path "/268c6120-58cb-44fb-87db-b7827ba409a7"
+					(reference "J1")
+					(unit 1)
+				)
+			)
+		)
+	)
+	(symbol
 		(lib_id "Personal_Library:RP2040-PICO")
 		(at 250.19 55.88 0)
@@
 					(unit 1)
 				)
+			)
+		)
+	)
+	(symbol
+		(lib_id "power:GND")
+		(at 48.26 43.18 0)
+		(mirror x)
+		(unit 1)
+		(body_style 1)
+		(exclude_from_sim no)
+		(in_bom yes)
+		(on_board yes)
+		(in_pos_files yes)
+		(dnp no)
+		(property "Reference" "#PWR021"
+			(at 48.26 36.83 0)
+			(hide yes)
+			(show_name no)
+			(do_not_autoplace no)
+			(effects
+				(font
+					(size 1.27 1.27)
+				)
+			)
+		)
+		(property "Value" "GND"
+			(at 48.26 38.1 0)
+			(show_name no)
+			(do_not_autoplace no)
+			(effects
+				(font
+					(size 1.27 1.27)
+				)
+			)
+		)
+		(property "Footprint" ""
+			(at 48.26 43.18 0)
+			(hide yes)
+			(show_name no)
+			(do_not_autoplace no)
+			(effects
+				(font
+					(size 1.27 1.27)
+				)
+			)
+		)
+		(property "Datasheet" ""
+			(at 48.26 43.18 0)
+			(hide yes)
+			(show_name no)
+			(do_not_autoplace no)
+			(effects
+				(font
+					(size 1.27 1.27)
+				)
+			)
+		)
+		(property "Description" "Power symbol creates a global label with name \"GND\" , ground"
+			(at 48.26 43.18 0)
+			(hide yes)
+			(show_name no)
+			(do_not_autoplace no)
+			(effects
+				(font
+					(size 1.27 1.27)
+				)
+			)
+		)
+		(pin "1"
+		)
+		(instances
+			(project "photoacoustic-detector"
+				(path "/268c6120-58cb-44fb-87db-b7827ba409a7"
+					(reference "#PWR021")
+					(unit 1)
+				)
